Commit message: limites robot1 actualizados

File: Proyecto_Final_ws/src/robot1_description/urdf/robot1.urdf (robot description, URDF)
Before this commit: robot robot1_xy, 4 links, 3 joints
Joints:
- joint arm_joint_r1: limit lower=-3.14 upper=3.14 effort=10.0 velocity=3.14 -> lower=-1.57 upper=1.57 effort=10.0 velocity=1.57
- joint forearm_joint_r1: limit lower=-3.14 upper=3.14 effort=10.0 velocity=3.14 -> lower=-1.57 upper=1.57 effort=10.0 velocity=1.57
