Commit message: Agrega cambios a archivos del robot 2

File: Proyecto_Final_ws/src/robot2_description/urdf/robot2.urdf (robot description, URDF)
Before this commit: robot robot2_rrr, 4 links, 3 joints
Joints:
- joint arm_joint_r2: limit lower=-1.57 upper=1.57 effort=10.0 velocity=3.14 -> lower=-3.14 upper=3.14 effort=10.0 velocity=3.14
- joint shoulder_joint_r2: limit lower=0 upper=1.57 effort=10.0 velocity=3.14 -> lower=-3.14 upper=3.14 effort=10.0 velocity=3.14

Commit message: archivos de robot2 actualizados y modificaciones de configuración.

File: Proyecto_Final_ws/src/robot2_description/urdf/robot2.urdf (robot description, URDF)
Before this commit: robot robot2_rrr, 4 links, 3 joints
Joints:
- joint arm_joint_r2: limit lower=-3.14 upper=3.14 effort=10.0 velocity=3.14 -> lower=-1.57 upper=1.57 effort=10.0 velocity=1.57
- joint shoulder_joint_r2: limit lower=-3.14 upper=3.14 effort=10.0 velocity=3.14 -> lower=0 upper=1.57 effort=10.0 velocity=1.57
